File: eagle/ms20_vcf.sch (EAGLE design)
At the start: 41 parts, among them IC1 LM13700N, IC2 TL082P, IC3 TL082P, Q1 BC559C, Q2 BC559C

Commit message: routed
Parts:
- C7: device rcl:CPOL-EUB45181A -> rcl:CPOL-EUB45181B
Changed lines of the file:
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@@
 <grid distance="0.1" unitdist="inch" unit="inch" style="lines" multiple="1" display="no" altdistance="0.01" altunitdist="inch" altunit="inch"/>
 <layers>
-<layer number="1" name="Top" color="4" fill="1" visible="no" active="no"/>
-<layer number="16" name="Bottom" color="1" fill="1" visible="no" active="no"/>
-<layer number="17" name="Pads" color="2" fill="1" visible="no" active="no"/>
-<layer number="18" name="Vias" color="2" fill="1" visible="no" active="no"/>
-<layer number="19" name="Unrouted" color="6" fill="1" visible="no" active="no"/>
-<layer number="20" name="Dimension" color="15" fill="1" visible="no" active="no"/>
-<layer number="21" name="tPlace" color="7" fill="1" visible="no" active="no"/>
-<layer number="22" name="bPlace" color="7" fill="1" visible="no" active="no"/>
-<layer number="23" name="tOrigins" color="15" fill="1" visible="no" active="no"/>
-<layer number="24" name="bOrigins" color="15" fill="1" visible="no" active="no"/>
-<layer number="25" name="tNames" color="7" fill="1" visible="no" active="no"/>
-<layer number="26" name="bNames" color="7" fill="1" visible="no" active="no"/>
-<layer number="27" name="tValues" color="7" fill="1" visible="no" active="no"/>
-<layer number="28" name="bValues" color="7" fill="1" visible="no" active="no"/>
+<layer number="1" name="Top" color="4" fill="1" visible="yes" active="no"/>
+<layer number="16" name="Bottom" color="1" fill="1" visible="yes" active="no"/>
+<layer number="17" name="Pads" color="2" fill="1" visible="yes" active="no"/>
+<layer number="18" name="Vias" color="2" fill="1" visible="yes" active="no"/>
+<layer number="19" name="Unrouted" color="6" fill="1" visible="yes" active="no"/>
+<layer number="20" name="Dimension" color="15" fill="1" visible="yes" active="no"/>
+<layer number="21" name="tPlace" color="7" fill="1" visible="yes" active="no"/>
+<layer number="22" name="bPlace" color="7" fill="1" visible="yes" active="no"/>
+<layer number="23" name="tOrigins" color="15" fill="1" visible="yes" active="no"/>
+<layer number="24" name="bOrigins" color="15" fill="1" visible="yes" active="no"/>
+<layer number="25" name="tNames" color="7" fill="1" visible="yes" active="no"/>
+<layer number="26" name="bNames" color="7" fill="1" visible="yes" active="no"/>
+<layer number="27" name="tValues" color="7" fill="1" visible="yes" active="no"/>
+<layer number="28" name="bValues" color="7" fill="1" visible="yes" active="no"/>
 <layer number="29" name="tStop" color="7" fill="3" visible="no" active="no"/>
 <layer number="30" name="bStop" color="7" fill="6" visible="no" active="no"/>
@@
 <layer number="35" name="tGlue" color="7" fill="4" visible="no" active="no"/>
 <layer number="36" name="bGlue" color="7" fill="5" visible="no" active="no"/>
-<layer number="37" name="tTest" color="7" fill="1" visible="no" active="no"/>
-<layer number="38" name="bTest" color="7" fill="1" visible="no" active="no"/>
+<layer number="37" name="tTest" color="7" fill="1" visible="yes" active="no"/>
+<layer number="38" name="bTest" color="7" fill="1" visible="yes" active="no"/>
 <layer number="39" name="tKeepout" color="4" fill="11" visible="no" active="no"/>
 <layer number="40" name="bKeepout" color="1" fill="11" visible="no" active="no"/>
@@
 <layer number="44" name="Drills" color="7" fill="1" visible="no" active="no"/>
 <layer number="45" name="Holes" color="7" fill="1" visible="no" active="no"/>
-<layer number="46" name="Milling" color="3" fill="1" visible="no" active="no"/>
-<layer number="47" name="Measures" color="7" fill="1" visible="no" active="no"/>
-<layer number="48" name="Document" color="7" fill="1" visible="no" active="no"/>
-<layer number="49" name="Reference" color="7" fill="1" visible="no" active="no"/>
-<layer number="50" name="dxf" color="7" fill="1" visible="no" active="no"/>
-<layer number="51" name="tDocu" color="7" fill="1" visible="no" active="no"/>
-<layer number="52" name="bDocu" color="7" fill="1" visible="no" active="no"/>
-<layer number="53" name="tGND_GNDA" color="7" fill="9" visible="no" active="no"/>
-<layer number="54" name="bGND_GNDA" color="1" fill="9" visible="no" active="no"/>
-<layer number="56" name="wert" color="7" fill="1" visible="no" active="no"/>
-<layer number="57" name="tCAD" color="7" fill="1" visible="no" active="no"/>
+<layer number="46" name="Milling" color="3" fill="1" visible="yes" active="no"/>
+<layer number="47" name="Measures" color="7" fill="1" visible="yes" active="no"/>
+<layer number="48" name="Document" color="7" fill="1" visible="yes" active="no"/>
+<layer number="49" name="Reference" color="7" fill="1" visible="yes" active="no"/>
+<layer number="50" name="dxf" color="7" fill="1" visible="yes" active="no"/>
+<layer number="51" name="tDocu" color="7" fill="1" visible="yes" active="no"/>
+<layer number="52" name="bDocu" color="7" fill="1" visible="yes" active="no"/>
+<layer number="53" name="tGND_GNDA" color="7" fill="9" visible="yes" active="no"/>
+<layer number="54" name="bGND_GNDA" color="1" fill="9" visible="yes" active="no"/>
+<layer number="56" name="wert" color="7" fill="1" visible="yes" active="no"/>
+<layer number="57" name="tCAD" color="7" fill="1" visible="yes" active="no"/>
 <layer number="90" name="Modules" color="5" fill="1" visible="no" active="yes"/>
 <layer number="91" name="Nets" color="2" fill="1" visible="yes" active="yes"/>
@@
 <part name="R18" library="rcl" deviceset="R-US_" device="0207/10" value="10k"/>
 <part name="R19" library="rcl" deviceset="R-US_" device="0207/10" value="10k"/>
-<part name="C7" library="rcl" deviceset="CPOL-EU" device="B45181A" value="0.47uF"/>
+<part name="C7" library="rcl" deviceset="CPOL-EU" device="B45181B" value="0.47uF"/>
 <part name="FREQ" library="pot" deviceset="3RP/1610N" device="" value="100k"/>
 <part name="R21" library="rcl" deviceset="R-US_" device="0207/10" value="100k"/>

Commit message: began changes for itead
Parts:
- removed C1, C2: 10uF, rcl:CPOL-USB45181A
- removed CV_2: AUDIO-JACK, erthenvar:AUDIO-JACK
- removed U$1: POWER, eurorack:POWER
- added C22, C23: 10u, rcl:CPOL-USB45181A
- added C24, C25: 100n, rcl:C-US050-024X044
- added CV2: (no value), con-phoenix-254:MPT2
- added FB3, FB4: FB, adafruit:FB
- added U2: POWER, eurorack:POWER
- C7: device rcl:CPOL-EUB45181B -> rcl:CPOL-EUB45181A
- CV2_LEV: device pot:3RP/1610N -> con-phoenix-254:MPT3
- CV_1, HP_IN, LP_IN, OUT: value AUDIO-JACK -> AUDIO-JACKITEAD; device erthenvar:AUDIO-JACK -> erthenvar:AUDIO-JACKITEAD
- Q1, Q2: value BC559C -> 2N3906; device transistor-pnp:BC559C -> transistor-pnp:2N3906
Connections:
- new net N$41: FB3.1, U2.+12V
- new net N$68: FB4.1, U2.-12V
- net +12V: now also C22.+, C24.1, FB3.2; no longer C1.+, U$1.+12V
- net -12V: now also C23.-, C25.2, FB4.2; no longer C2.-, U$1.-12V
- net GND: now also C22.-, C23.+, C24.2, C25.1, CV2-2.1, CV2_LEV-3.1, U2.GND; no longer C1.-, C2.+, CV2_LEV.A, CV_2.RING, U$1.GND
- net N$23: now also CV2-1.1, CV2_LEV-1.1; no longer CV2_LEV.E, CV_2.TIP
- net N$27: now also U2.CV; no longer U$1.CV
- net N$8: now also CV2_LEV-2.1; no longer CV2_LEV.S

Commit message: decoupling caps
Parts:
- added C1, C10, C2, C4, C8, C9: 100n, rcl:C-USC1206
Connections:
- net +12V: now also C1.1, C2.1, C4.1
- net -12V: now also C10.2, C8.2, C9.2
- net GND: now also C1.2, C10.1, C2.2, C4.2, C8.1, C9.1
Changed lines of the file:
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@@
 <part name="C25" library="rcl" deviceset="C-US" device="050-024X044" value="100n"/>
 <part name="GND1" library="supply1" deviceset="GND" device=""/>
+<part name="C1" library="rcl" deviceset="C-US" device="C1206" value="100n"/>
+<part name="C2" library="rcl" deviceset="C-US" device="C1206" value="100n"/>
+<part name="C4" library="rcl" deviceset="C-US" device="C1206" value="100n"/>
+<part name="C8" library="rcl" deviceset="C-US" device="C1206" value="100n"/>
+<part name="C9" library="rcl" deviceset="C-US" device="C1206" value="100n"/>
+<part name="C10" library="rcl" deviceset="C-US" device="C1206" value="100n"/>
+<part name="GND14" library="supply1" deviceset="GND" device=""/>
 </parts>
 <sheets>
@@
 </instance>
 <instance part="GND1" gate="1" x="167.64" y="83.82"/>
+<instance part="C1" gate="G$1" x="180.34" y="81.28"/>
+<instance part="C2" gate="G$1" x="193.04" y="81.28"/>
+<instance part="C4" gate="G$1" x="210.82" y="81.28"/>
+<instance part="C8" gate="G$1" x="210.82" y="66.04"/>
+<instance part="C9" gate="G$1" x="193.04" y="66.04"/>
+<instance part="C10" gate="G$1" x="180.34" y="66.04"/>
+<instance part="GND14" gate="1" x="223.52" y="55.88"/>
 </instances>
 <busses>
@@
 <pinref part="P-1" gate="1" pin="-12V"/>
 <pinref part="IC1" gate="G$5" pin="V-"/>
-<wire x1="203.835" y1="57.15" x2="187.96" y2="53.34" width="0.1524" layer="91"/>
+<wire x1="203.835" y1="57.15" x2="205.74" y2="57.15" width="0.1524" layer="91"/>
+<wire x1="205.74" y1="57.15" x2="205.74" y2="53.34" width="0.1524" layer="91"/>
+<wire x1="205.74" y1="53.34" x2="193.04" y2="53.34" width="0.1524" layer="91"/>
 <pinref part="IC2" gate="P" pin="V-"/>
+<wire x1="193.04" y1="53.34" x2="187.96" y2="53.34" width="0.1524" layer="91"/>
 <wire x1="187.96" y1="66.04" x2="187.96" y2="55.88" width="0.1524" layer="91"/>
 <junction x="187.96" y="53.34"/>
@@
 <wire x1="187.96" y1="55.88" x2="187.96" y2="53.34" width="0.1524" layer="91"/>
 <wire x1="172.72" y1="66.04" x2="172.72" y2="55.88" width="0.1524" layer="91"/>
-<wire x1="172.72" y1="55.88" x2="187.96" y2="55.88" width="0.1524" layer="91"/>
+<wire x1="172.72" y1="55.88" x2="180.34" y2="55.88" width="0.1524" layer="91"/>
 <junction x="187.96" y="55.88"/>
+<pinref part="C8" gate="G$1" pin="2"/>
+<wire x1="180.34" y1="55.88" x2="187.96" y2="55.88" width="0.1524" layer="91"/>
+<wire x1="205.74" y1="53.34" x2="210.82" y2="53.34" width="0.1524" layer="91"/>
+<wire x1="210.82" y1="53.34" x2="210.82" y2="60.96" width="0.1524" layer="91"/>
+<junction x="205.74" y="53.34"/>
+<pinref part="C9" gate="G$1" pin="2"/>
+<wire x1="193.04" y1="60.96" x2="193.04" y2="53.34" width="0.1524" layer="91"/>
+<junction x="193.04" y="53.34"/>
+<pinref part="C10" gate="G$1" pin="2"/>
+<wire x1="180.34" y1="60.96" x2="180.34" y2="55.88" width="0.1524" layer="91"/>
+<junction x="180.34" y="55.88"/>
 </segment>
 <segment>
@@
 <pinref part="P+1" gate="1" pin="+12V"/>
 <pinref part="IC1" gate="G$5" pin="V+"/>
-<wire x1="203.835" y1="86.36" x2="187.96" y2="93.98" width="0.1524" layer="91"/>
+<wire x1="203.835" y1="86.36" x2="203.2" y2="86.36" width="0.1524" layer="91"/>
+<wire x1="203.2" y1="86.36" x2="203.2" y2="93.98" width="0.1524" layer="91"/>
+<wire x1="203.2" y1="93.98" x2="193.04" y2="93.98" width="0.1524" layer="91"/>
 <pinref part="IC2" gate="P" pin="V+"/>
+<wire x1="193.04" y1="93.98" x2="187.96" y2="93.98" width="0.1524" layer="91"/>
 <wire x1="187.96" y1="81.28" x2="187.96" y2="86.36" width="0.1524" layer="91"/>
 <junction x="187.96" y="93.98"/>
@@
 <wire x1="187.96" y1="86.36" x2="187.96" y2="93.98" width="0.1524" layer="91"/>
 <wire x1="172.72" y1="81.28" x2="172.72" y2="86.36" width="0.1524" layer="91"/>
-<wire x1="172.72" y1="86.36" x2="187.96" y2="86.36" width="0.1524" layer="91"/>
+<wire x1="172.72" y1="86.36" x2="180.34" y2="86.36" width="0.1524" layer="91"/>
 <junction x="187.96" y="86.36"/>
+<pinref part="C4" gate="G$1" pin="1"/>
+<wire x1="180.34" y1="86.36" x2="187.96" y2="86.36" width="0.1524" layer="91"/>
+<wire x1="203.2" y1="93.98" x2="210.82" y2="93.98" width="0.1524" layer="91"/>
+<wire x1="210.82" y1="93.98" x2="210.82" y2="83.82" width="0.1524" layer="91"/>
+<junction x="203.2" y="93.98"/>
+<pinref part="C1" gate="G$1" pin="1"/>
+<wire x1="180.34" y1="86.36" x2="180.34" y2="83.82" width="0.1524" layer="91"/>
+<junction x="180.34" y="86.36"/>
+<pinref part="C2" gate="G$1" pin="1"/>
+<wire x1="193.04" y1="83.82" x2="193.04" y2="93.98" width="0.1524" layer="91"/>
+<junction x="193.04" y="93.98"/>
 </segment>
 <segment>
@@
 <pinref part="U2" gate="G$1" pin="GND"/>
 </segment>
+<segment>
+<pinref part="GND14" gate="1" pin="GND"/>
+<wire x1="180.34" y1="73.66" x2="193.04" y2="73.66" width="0.1524" layer="91"/>
+<wire x1="193.04" y1="73.66" x2="210.82" y2="73.66" width="0.1524" layer="91"/>
+<wire x1="210.82" y1="73.66" x2="223.52" y2="73.66" width="0.1524" layer="91"/>
+<wire x1="223.52" y1="73.66" x2="223.52" y2="58.42" width="0.1524" layer="91"/>
+<pinref part="C1" gate="G$1" pin="2"/>
+<wire x1="180.34" y1="76.2" x2="180.34" y2="73.66" width="0.1524" layer="91"/>
+<pinref part="C10" gate="G$1" pin="1"/>
+<wire x1="180.34" y1="68.58" x2="180.34" y2="73.66" width="0.1524" layer="91"/>
+<junction x="180.34" y="73.66"/>
+<pinref part="C2" gate="G$1" pin="2"/>
+<wire x1="193.04" y1="76.2" x2="193.04" y2="73.66" width="0.1524" layer="91"/>
+<junction x="193.04" y="73.66"/>
+<pinref part="C9" gate="G$1" pin="1"/>
+<wire x1="193.04" y1="68.58" x2="193.04" y2="73.66" width="0.1524" layer="91"/>
+<pinref part="C4" gate="G$1" pin="2"/>
+<wire x1="210.82" y1="76.2" x2="210.82" y2="73.66" width="0.1524" layer="91"/>
+<junction x="210.82" y="73.66"/>
+<pinref part="C8" gate="G$1" pin="1"/>
+<wire x1="210.82" y1="68.58" x2="210.82" y2="73.66" width="0.1524" layer="91"/>
+</segment>
 </net>
 <net name="N$7" class="0">
@@
 <wire x1="-5.08" y1="96.52" x2="-2.54" y2="96.52" width="0.1524" layer="91"/>
 <wire x1="-2.54" y1="96.52" x2="-2.54" y2="104.14" width="0.1524" layer="91"/>
-<wire x1="-2.54" y1="104.14" x2="109.22" y2="104.14" width="0.1524" layer="91"/>
-<wire x1="109.22" y1="104.14" x2="109.22" y2="71.12" width="0.1524" layer="91"/>
+<wire x1="-2.54" y1="104.14" x2="106.68" y2="104.14" width="0.1524" layer="91"/>
+<wire x1="106.68" y1="104.14" x2="106.68" y2="71.12" width="0.1524" layer="91"/>
 <pinref part="U2" gate="G$1" pin="CV"/>
 <wire x1="127" y1="83.82" x2="137.16" y2="83.82" width="0.1524" layer="91"/>
-<wire x1="109.22" y1="71.12" x2="137.16" y2="71.12" width="0.1524" layer="91"/>
+<wire x1="106.68" y1="71.12" x2="137.16" y2="71.12" width="0.1524" layer="91"/>
 <wire x1="137.16" y1="71.12" x2="137.16" y2="83.82" width="0.1524" layer="91"/>
 </segment>

Commit message: parts on the board
Parts:
- R1, R10, R11, R12, R13, R14, R15, R16, R17, R18, R19, R21, R4, R5, R6, R7, R8, R9: device rcl:R-US_0207/10 -> rcl:R-US_0207/7
Changed lines of the file:
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@@
 <part name="IC2" library="linear" deviceset="TL082" device="P"/>
 <part name="IC3" library="linear" deviceset="TL082" device="P"/>
-<part name="R1" library="rcl" deviceset="R-US_" device="0207/10" value="100k"/>
+<part name="R1" library="rcl" deviceset="R-US_" device="0207/7" value="100k"/>
 <part name="CV1_LEV" library="pot" deviceset="3RP/1610N" device="" value="100k"/>
 <part name="P+1" library="supply1" deviceset="+12V" device=""/>
@@
 <part name="Q1" library="transistor-pnp" deviceset="2N3906" device=""/>
 <part name="Q2" library="transistor-pnp" deviceset="2N3906" device=""/>
-<part name="R4" library="rcl" deviceset="R-US_" device="0207/10" value="10k"/>
+<part name="R4" library="rcl" deviceset="R-US_" device="0207/7" value="10k"/>
 <part name="LED1" library="led" deviceset="LED" device="5MM" value="green"/>
 <part name="LED2" library="led" deviceset="LED" device="5MM" value="green"/>
-<part name="R5" library="rcl" deviceset="R-US_" device="0207/10" value="1k8"/>
+<part name="R5" library="rcl" deviceset="R-US_" device="0207/7" value="1k8"/>
 <part name="RESONANCE" library="pot" deviceset="3RP/1610N" device="" value="100k"/>
-<part name="R7" library="rcl" deviceset="R-US_" device="0207/10" value="4k7"/>
+<part name="R7" library="rcl" deviceset="R-US_" device="0207/7" value="4k7"/>
 <part name="C3" library="rcl" deviceset="C-US" device="050-024X044" value="4n7"/>
-<part name="R8" library="rcl" deviceset="R-US_" device="0207/10" value="470k"/>
+<part name="R8" library="rcl" deviceset="R-US_" device="0207/7" value="470k"/>
 <part name="P-2" library="supply1" deviceset="-12V" device=""/>
 <part name="GND2" library="supply1" deviceset="GND" device=""/>
-<part name="R9" library="rcl" deviceset="R-US_" device="0207/10" value="100k"/>
+<part name="R9" library="rcl" deviceset="R-US_" device="0207/7" value="100k"/>
 <part name="GND4" library="supply1" deviceset="GND" device=""/>
 <part name="GND5" library="supply1" deviceset="GND" device=""/>
-<part name="R6" library="rcl" deviceset="R-US_" device="0207/10" value="1k8"/>
+<part name="R6" library="rcl" deviceset="R-US_" device="0207/7" value="1k8"/>
 <part name="GND6" library="supply1" deviceset="GND" device=""/>
-<part name="R10" library="rcl" deviceset="R-US_" device="0207/10" value="220"/>
+<part name="R10" library="rcl" deviceset="R-US_" device="0207/7" value="220"/>
 <part name="GND7" library="supply1" deviceset="GND" device=""/>
-<part name="R11" library="rcl" deviceset="R-US_" device="0207/10" value="220"/>
+<part name="R11" library="rcl" deviceset="R-US_" device="0207/7" value="220"/>
 <part name="GND8" library="supply1" deviceset="GND" device=""/>
 <part name="GND9" library="supply1" deviceset="GND" device=""/>
 <part name="C5" library="rcl" deviceset="C-US" device="050-024X044" value="1n"/>
 <part name="C6" library="rcl" deviceset="C-US" device="050-024X044" value="1n"/>
-<part name="R12" library="rcl" deviceset="R-US_" device="0207/10" value="10k"/>
-<part name="R13" library="rcl" deviceset="R-US_" device="0207/10" value="10k"/>
-<part name="R14" library="rcl" deviceset="R-US_" device="0207/10" value="10k"/>
-<part name="R15" library="rcl" deviceset="R-US_" device="0207/10" value="220"/>
+<part name="R12" library="rcl" deviceset="R-US_" device="0207/7" value="10k"/>
+<part name="R13" library="rcl" deviceset="R-US_" device="0207/7" value="10k"/>
+<part name="R14" library="rcl" deviceset="R-US_" device="0207/7" value="10k"/>
+<part name="R15" library="rcl" deviceset="R-US_" device="0207/7" value="220"/>
 <part name="GND10" library="supply1" deviceset="GND" device=""/>
-<part name="R16" library="rcl" deviceset="R-US_" device="0207/10" value="220"/>
+<part name="R16" library="rcl" deviceset="R-US_" device="0207/7" value="220"/>
 <part name="GND11" library="supply1" deviceset="GND" device=""/>
 <part name="GND12" library="supply1" deviceset="GND" device=""/>
-<part name="R17" library="rcl" deviceset="R-US_" device="0207/10" value="10k"/>
+<part name="R17" library="rcl" deviceset="R-US_" device="0207/7" value="10k"/>
 <part name="GND13" library="supply1" deviceset="GND" device=""/>
-<part name="R18" library="rcl" deviceset="R-US_" device="0207/10" value="10k"/>
-<part name="R19" library="rcl" deviceset="R-US_" device="0207/10" value="10k"/>
+<part name="R18" library="rcl" deviceset="R-US_" device="0207/7" value="10k"/>
+<part name="R19" library="rcl" deviceset="R-US_" device="0207/7" value="10k"/>
 <part name="C7" library="rcl" deviceset="CPOL-EU" device="B45181A" value="0.47uF"/>
 <part name="FREQ" library="pot" deviceset="3RP/1610N" device="" value="100k"/>
-<part name="R21" library="rcl" deviceset="R-US_" device="0207/10" value="100k"/>
+<part name="R21" library="rcl" deviceset="R-US_" device="0207/7" value="100k"/>
 <part name="P+3" library="supply1" deviceset="+12V" device=""/>
 <part name="P-4" library="supply1" deviceset="-12V" device=""/>
