File: eagle/ms20_vcf.brd (EAGLE design)
At the start: 100 x 80 mm, 41 parts, among them IC1 LM13700N, IC2 TL082P, IC3 TL082P, Q1 BC559C, Q2 BC559C

Commit message: toward routes
Parts:
- moved R12 55.3 mm to (12.7, 26.7), turned to 90 degrees
- moved R15 43.0 mm to (76.2, 54.6), turned to 180 degrees
- moved R16 41.1 mm to (76.2, 50.8), turned to 180 degrees
- moved IC3 40.1 mm to (72.4, 24.1)
- moved R5 38.2 mm to (69.8, 14.0)
- moved LED1 36.4 mm to (82.5, 25.4), turned to 0 degrees
- moved R8 35.3 mm to (54.6, 29.2)
- moved IC2 31.4 mm to (47.0, 43.2), turned to 0 degrees
- moved C5 29.5 mm to (86.4, 40.6), turned to 0 degrees
- moved R4 29.5 mm to (90.2, 30.5)
- moved R19 29.0 mm to (45.7, 67.3), turned to 0 degrees
- moved LED2 28.0 mm to (82.5, 33.0), turned to 180 degrees
- moved R18 27.2 mm to (45.7, 63.5), turned to 180 degrees
- moved CV2_LEV 27.2 mm to (25.4, 41.9), turned to 0 degrees
- moved R6 27.1 mm to (49.5, 29.2), turned to 270 degrees
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Routing:
- net GND: track 340.1 -> 0.00 mm
- net -12V: track 223.6 -> 0.00 mm
- net +12V: track 215.9 -> 0.00 mm
- net N$11: track 155.9 -> 0.00 mm
- net N$10: track 146.1 -> 0.00 mm
- net N$9: track 102.8 -> 0.00 mm, vias 2 -> 0
- net N$6: track 101.1 -> 0.00 mm
- net N$3: track 97.7 -> 0.00 mm
- net N$25: track 96.8 -> 0.00 mm
- net N$19: track 83.3 -> 0.00 mm
- net N$5: track 62.9 -> 0.00 mm
- net N$21: track 40.0 -> 0.00 mm
- net N$2: track 34.4 -> 0.00 mm
- net N$1: track 29.1 -> 0.00 mm
- net N$17: track 25.1 -> 0.00 mm
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
Commit message: routed
Parts:
- C7: device rcl:B45181A -> rcl:B45181B
- moved C6 60.0 mm to (64.8, 27.9)
- moved R5 41.5 mm to (86.4, 52.1), turned to 270 degrees
- moved HP_IN 39.5 mm to (49.5, 2.54)
- moved CV_2 28.5 mm to (6.35, 50.8), turned to 0 degrees
- moved R19 26.7 mm to (72.4, 68.6), turned to 270 degrees
- moved CV1_LEV 25.5 mm to (19.1, 6.35)
- moved CV_1 24.3 mm to (10.2, 2.54)
- moved R1 23.4 mm to (19.1, 19.1)
- moved R12 22.2 mm to (31.8, 38.1)
- moved RESONANCE 21.7 mm to (58.4, 6.35)
- moved R18 19.3 mm to (63.5, 71.1), turned to 0 degrees
- moved LP_IN 16.7 mm to (38.1, 2.54)
- moved R4 14.9 mm to (85.1, 44.5), turned to 0 degrees
- moved FREQ 14.2 mm to (76.2, 6.35)
- moved C2 14.2 mm to (17.8, 59.7), turned to 180 degrees
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Routing:
- net GND: track 0.00 -> 436.4 mm
- net +12V: track 0.00 -> 187.1 mm
- net -12V: track 0.00 -> 135.9 mm
- net N$16: track 0.00 -> 95.5 mm, vias 0 -> 2
- net N$27: track 0.00 -> 80.1 mm, vias 0 -> 2
- net N$21: track 0.00 -> 65.5 mm
- net N$14: track 0.00 -> 60.4 mm
- net N$6: track 0.00 -> 47.9 mm
- net N$9: track 0.00 -> 41.5 mm, vias 0 -> 4
- net N$12: track 0.00 -> 40.0 mm, vias 0 -> 2
- net N$24: track 0.00 -> 38.2 mm
- net N$1: track 0.00 -> 35.1 mm
- net N$22: track 0.00 -> 35.1 mm
- net N$10: track 0.00 -> 32.8 mm
- net N$11: track 0.00 -> 30.5 mm
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
Commit message: rerouted and milling
Parts:
- moved R21 16.5 mm to (66.0, 21.6)
- moved R8 1.27 mm to (52.1, 40.6)
- moved R17 1.14 mm to (53.6, 65.3)
Routing:
- net N$22: track 35.1 -> 17.3 mm
- net N$21: track 65.5 -> 80.2 mm
- net N$26: track 22.8 -> 27.6 mm
- net -12V: track 135.9 -> 139.0 mm
- net N$16: track 95.5 -> 92.6 mm
- net N$6: track 47.9 -> 45.9 mm
- net N$19: track 16.8 -> 15.5 mm
- net N$10: track 32.8 -> 31.5 mm
- net +12V: track 187.1 -> 188.2 mm
- net N$4: track 21.5 -> 20.9 mm
Other:
- board size 100 x 80 mm -> 100.8 x 80 mm

Commit message: burned and works
Routing:
- net N$24: track 38.2 -> 34.7 mm
- net N$1: track 35.1 -> 33.6 mm
- net N$3: track 18.4 -> 19.3 mm
- net GND: track 436.7 -> 436.0 mm
Changed lines of the file:
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@@
 <wire x1="57.15" y1="52.07" x2="60.96" y2="53.34" width="0.8128" layer="16"/>
 <wire x1="57.15" y1="45.72" x2="57.15" y2="52.07" width="0.8128" layer="16"/>
-<wire x1="27.305" y1="46.355" x2="16.51" y2="59.69" width="0.8128" layer="16"/>
-<wire x1="27.305" y1="42.545" x2="27.305" y2="46.355" width="0.8128" layer="16"/>
-<wire x1="28.575" y1="40.005" x2="27.305" y2="42.545" width="0.8128" layer="16"/>
-<wire x1="33.655" y1="40.005" x2="28.575" y2="40.005" width="0.8128" layer="16"/>
+<wire x1="17.145" y1="55.245" x2="16.51" y2="59.69" width="0.8128" layer="16"/>
+<wire x1="24.765" y1="51.435" x2="17.145" y2="55.245" width="0.8128" layer="16"/>
+<wire x1="29.845" y1="40.005" x2="24.765" y2="51.435" width="0.8128" layer="16"/>
+<wire x1="33.655" y1="40.005" x2="29.845" y2="40.005" width="0.8128" layer="16"/>
 <wire x1="36.195" y1="49.53" x2="33.655" y2="40.005" width="0.8128" layer="16"/>
 <wire x1="46.99" y1="49.53" x2="36.195" y2="49.53" width="0.8128" layer="16"/>
@@
 <wire x1="85.09" y1="29.21" x2="85.09" y2="27.305" width="0.8128" layer="16"/>
 <wire x1="85.09" y1="29.21" x2="85.09" y2="35.56" width="0.8128" layer="16"/>
-<wire x1="85.09" y1="35.56" x2="85.09" y2="41.91" width="0.8128" layer="16"/>
-<wire x1="85.09" y1="41.91" x2="87.63" y2="44.45" width="0.8128" layer="16"/>
-<wire x1="87.63" y1="44.45" x2="90.17" y2="44.45" width="0.8128" layer="16"/>
+<wire x1="85.09" y1="35.56" x2="85.09" y2="39.37" width="0.8128" layer="16"/>
+<wire x1="85.09" y1="39.37" x2="90.17" y2="44.45" width="0.8128" layer="16"/>
 </signal>
 <signal name="N$2">
@@
 <wire x1="43.18" y1="45.72" x2="43.18" y2="41.91" width="0.8128" layer="16"/>
 <wire x1="43.18" y1="41.91" x2="46.99" y2="40.64" width="0.8128" layer="16"/>
-<wire x1="48.895" y1="34.925" x2="48.26" y2="34.29" width="0.6604" layer="16"/>
-<wire x1="48.895" y1="40.005" x2="48.895" y2="34.925" width="0.8128" layer="16"/>
-<wire x1="46.99" y1="40.64" x2="48.895" y2="40.005" width="0.8128" layer="16"/>
+<wire x1="49.403" y1="34.417" x2="48.26" y2="34.29" width="0.6604" layer="16"/>
+<wire x1="49.403" y1="39.497" x2="49.403" y2="34.417" width="0.8128" layer="16"/>
+<wire x1="46.99" y1="40.64" x2="49.403" y2="39.497" width="0.8128" layer="16"/>
 </signal>
 <signal name="N$4">
@@
 <wire x1="73.787" y1="75.819" x2="79.375" y2="70.485" width="0.8128" layer="16"/>
 <wire x1="36.957" y1="75.819" x2="73.787" y2="75.819" width="0.8128" layer="16"/>
-<wire x1="50.8" y1="33.02" x2="54.61" y2="31.75" width="0.8128" layer="16"/>
-<wire x1="50.8" y1="40.64" x2="50.8" y2="38.1" width="0.8128" layer="16"/>
-<wire x1="50.8" y1="38.1" x2="50.8" y2="33.02" width="0.8128" layer="16"/>
-<wire x1="45.72" y1="45.72" x2="50.8" y2="40.64" width="0.8128" layer="16"/>
-<wire x1="50.8" y1="38.1" x2="57.15" y2="38.1" width="0.8128" layer="16"/>
+<wire x1="52.07" y1="33.02" x2="54.61" y2="31.75" width="0.8128" layer="16"/>
+<wire x1="51.054" y1="42.164" x2="51.816" y2="38.1" width="0.8128" layer="16"/>
+<wire x1="51.816" y1="38.1" x2="52.07" y2="33.02" width="0.8128" layer="16"/>
+<wire x1="45.72" y1="45.72" x2="46.99" y2="43.18" width="0.8128" layer="16"/>
+<wire x1="46.99" y1="43.18" x2="47.498" y2="42.926" width="0.8128" layer="16"/>
+<wire x1="47.498" y1="42.926" x2="51.054" y2="42.164" width="0.8128" layer="16"/>
+<wire x1="51.816" y1="38.1" x2="57.15" y2="38.1" width="0.8128" layer="16"/>
 <wire x1="17.145" y1="3.81" x2="14.605" y2="6.35" width="0.8128" layer="16"/>
 <wire x1="50.8" y1="3.81" x2="44.45" y2="3.81" width="0.8128" layer="16"/>
@@
 <contactref element="IC2" pad="5"/>
 <contactref element="C5" pad="1"/>
-<wire x1="60.96" y1="55.88" x2="62.23" y2="55.88" width="0.6096" layer="16"/>
+<wire x1="60.96" y1="55.88" x2="62.23" y2="55.88" width="0.8128" layer="16"/>
 <wire x1="62.23" y1="55.88" x2="63.754" y2="54.61" width="0.8128" layer="16"/>
 <wire x1="63.754" y1="54.61" x2="63.754" y2="44.45" width="0.8128" layer="16"/>
-<via x="63.754" y="44.45" extent="1-16" drill="0.6" diameter="0.8128" shape="square"/>
+<via x="63.754" y="44.45" extent="1-16" drill="0.8" diameter="0.8128" shape="square"/>
 <wire x1="63.754" y1="44.45" x2="68.58" y2="44.45" width="0.8128" layer="1"/>
-<via x="68.58" y="44.45" extent="1-16" drill="0.6" diameter="0.8128" shape="square"/>
+<via x="68.58" y="44.45" extent="1-16" drill="0.8" diameter="0.8128" shape="square"/>
 <wire x1="60.96" y1="55.88" x2="57.15" y2="55.88" width="0.8128" layer="16"/>
-<via x="57.15" y="55.88" extent="1-16" drill="0.6" diameter="0.8128" shape="square"/>
+<via x="57.15" y="55.88" extent="1-16" drill="0.8" diameter="0.8128" shape="square"/>
 <wire x1="57.15" y1="55.88" x2="52.07" y2="55.88" width="0.8128" layer="1"/>
-<via x="52.07" y="55.88" extent="1-16" drill="0.6" diameter="0.8128" shape="square"/>
+<via x="52.07" y="55.88" extent="1-16" drill="0.8" diameter="0.8128" shape="square"/>
 <wire x1="52.07" y1="55.88" x2="48.26" y2="53.34" width="0.8128" layer="16"/>
 <wire x1="76.2" y1="46.99" x2="74.93" y2="48.26" width="0.8128" layer="16"/>
@@
 <wire x1="66.04" y1="31.75" x2="66.04" y2="54.61" width="0.8128" layer="16"/>
 <wire x1="66.04" y1="54.61" x2="67.31" y2="55.88" width="0.8128" layer="16"/>
-<wire x1="67.31" y1="55.88" x2="68.58" y2="55.88" width="0.6096" layer="16"/>
+<wire x1="67.31" y1="55.88" x2="68.58" y2="55.88" width="0.8128" layer="16"/>
 <wire x1="66.04" y1="31.75" x2="64.77" y2="30.48" width="0.8128" layer="16"/>
 <wire x1="68.58" y1="30.48" x2="64.77" y2="30.48" width="0.8128" layer="16"/>
@@
 <wire x1="63.42" y1="6.35" x2="63.42" y2="12.62" width="0.8128" layer="16"/>
 <wire x1="63.42" y1="12.62" x2="64.77" y2="13.97" width="0.8128" layer="16"/>
-<via x="64.77" y="13.97" extent="1-16" drill="0.6" diameter="0.8128" shape="square"/>
+<via x="64.77" y="13.97" extent="1-16" drill="0.8" diameter="0.8128" shape="square"/>
 <wire x1="64.77" y1="13.97" x2="82.55" y2="13.97" width="0.8128" layer="1"/>
-<via x="82.55" y="13.97" extent="1-16" drill="0.6" diameter="0.8128" shape="square"/>
+<via x="82.55" y="13.97" extent="1-16" drill="0.8" diameter="0.8128" shape="square"/>
 <wire x1="82.55" y1="13.97" x2="82.55" y2="18.415" width="0.8128" layer="16"/>
 <wire x1="82.55" y1="18.415" x2="81.915" y2="19.05" width="0.8128" layer="16"/>
@@
 <wire x1="45.72" y1="53.34" x2="43.18" y2="53.34" width="0.8128" layer="16"/>
 <wire x1="53.594" y1="60.198" x2="49.53" y2="60.96" width="0.8128" layer="16"/>
-<wire x1="46.355" y1="53.975" x2="45.72" y2="53.34" width="0.6604" layer="16"/>
-<wire x1="46.99" y1="57.785" x2="46.355" y2="53.975" width="0.8128" layer="16"/>
+<wire x1="45.593" y1="53.213" x2="45.72" y2="53.34" width="0.6604" layer="16"/>
+<wire x1="46.99" y1="57.785" x2="45.593" y2="53.213" width="0.8128" layer="16"/>
 <wire x1="49.53" y1="60.96" x2="46.99" y2="57.785" width="0.8128" layer="16"/>
 </signal>
@@
 <wire x1="78.486" y1="66.04" x2="78.486" y2="57.15" width="0.8128" layer="16"/>
 <wire x1="78.486" y1="57.15" x2="85.09" y2="52.07" width="0.8128" layer="16"/>
-<wire x1="85.09" y1="52.07" x2="88.9" y2="52.07" width="0.8128" layer="16"/>
-<via x="94.234" y="39.37" extent="1-16" drill="0.6" diameter="0.8128" shape="square"/>
+<wire x1="85.09" y1="52.07" x2="87.884" y2="52.07" width="0.8128" layer="16"/>
+<via x="94.234" y="39.37" extent="1-16" drill="0.8" diameter="0.8128" shape="square"/>
 <wire x1="94.234" y1="39.37" x2="62.23" y2="39.37" width="0.8128" layer="1"/>
-<via x="62.23" y="39.37" extent="1-16" drill="0.6" diameter="0.8128" shape="square"/>
+<via x="62.23" y="39.37" extent="1-16" drill="0.8" diameter="0.8128" shape="square"/>
 <wire x1="62.23" y1="39.37" x2="58.42" y2="34.29" width="0.8128" layer="16"/>
 <wire x1="58.42" y1="34.29" x2="54.61" y2="34.29" width="0.8128" layer="16"/>
-<wire x1="88.9" y1="52.07" x2="94.234" y2="46.228" width="0.8128" layer="16"/>
+<wire x1="87.884" y1="52.07" x2="94.234" y2="46.228" width="0.8128" layer="16"/>
 <wire x1="94.234" y1="46.228" x2="94.234" y2="39.37" width="0.8128" layer="16"/>
 <wire x1="73.66" y1="71.12" x2="73.66" y2="72.39" width="0.8128" layer="16"/>
@@
 <wire x1="24.05" y1="14.05" x2="20.32" y2="17.78" width="0.8128" layer="16"/>
 <wire x1="20.32" y1="17.78" x2="16.51" y2="17.78" width="0.8128" layer="16"/>
-<wire x1="16.51" y1="17.78" x2="12.7" y2="10.16" width="0.8128" layer="16"/>
-<wire x1="12.7" y1="10.16" x2="8.51" y2="10.16" width="0.8128" layer="16"/>
-<wire x1="8.51" y1="10.16" x2="5.16" y2="18.24" width="0.8128" layer="16"/>
+<wire x1="16.51" y1="17.78" x2="12.192" y2="12.192" width="0.8128" layer="16"/>
+<wire x1="12.192" y1="12.192" x2="8.002" y2="12.192" width="0.8128" layer="16"/>
+<wire x1="8.002" y1="12.192" x2="5.16" y2="18.24" width="0.8128" layer="16"/>
 </signal>
 <signal name="N$25">
@@
 <wire x1="31.75" y1="71.12" x2="31.75" y2="68.58" width="0.8128" layer="16"/>
 <wire x1="31.75" y1="68.58" x2="31.75" y2="64.77" width="0.8128" layer="16"/>
-<via x="31.75" y="64.77" extent="1-16" drill="0.6" diameter="0.8128" shape="square"/>
+<via x="31.75" y="64.77" extent="1-16" drill="0.8" diameter="0.8128" shape="square"/>
 <wire x1="31.75" y1="64.77" x2="15.24" y2="64.77" width="0.8128" layer="1"/>
 <wire x1="15.24" y1="64.77" x2="2.54" y2="52.07" width="0.8128" layer="1"/>
 <wire x1="2.54" y1="52.07" x2="2.54" y2="30.48" width="0.8128" layer="1"/>
 <wire x1="2.54" y1="30.48" x2="10.16" y2="22.86" width="0.8128" layer="1"/>
-<via x="10.16" y="22.86" extent="1-16" drill="0.6" diameter="0.8128" shape="square"/>
+<via x="10.16" y="22.86" extent="1-16" drill="0.8" diameter="0.8128" shape="square"/>
 <wire x1="10.16" y1="22.86" x2="10.16" y2="16.24" width="0.8128" layer="16"/>
 <wire x1="10.16" y1="16.24" x2="10.36" y2="16.04" width="0.8128" layer="16"/>

Commit message: began changes for itead
Parts:
- removed C1, C2: 10uF, rcl:B45181A
- removed CV_2: AUDIO-JACK, erthenvar:ERTHENVAR-JACK-90DEG
- removed U$1: POWER, eurorack:POWER_16
- added C22, C23: 10u, rcl:B45181A
- added C24, C25: 100n, rcl:C050-024X044
- added CV2: (no value), con-phoenix-254:2POL254
- added FB3, FB4: FB, adafruit:FB
- added U2: POWER, eurorack:POWER_16
- C7: device rcl:B45181B -> rcl:B45181A
- CV2_LEV: device pot:3RP/1610N -> con-phoenix-254:3POL254
- CV_1, HP_IN, LP_IN, OUT: value AUDIO-JACK -> AUDIO-JACKITEAD; device erthenvar:ERTHENVAR-JACK-90DEG -> erthenvar:JACK-90DEG-ITEAD
- Q1, Q2: value BC559C -> 2N3906; device transistor-pnp:TO92-EBC -> transistor-pnp:TO92
- moved CV2_LEV 17.3 mm to (6.35, 33.0), turned to 0 degrees
Connections:
- new net N$41: FB3.P$1, U2.10, U2.9
- new net N$68: FB4.P$1, U2.1, U2.2
- net +12V: now also C22.+, C24.1, FB3.P$2, FREQ.6; no longer C1.+, U$1.10, U$1.9
- net -12V: now also C23.-, C25.2, FB4.P$2, FREQ.4; no longer C2.-, U$1.1, U$1.2
- net GND: now also C22.-, C23.+, C24.2, C25.1, CV1_LEV.4, CV2.2, CV2_LEV.3, Q2.2, RESONANCE.4, U2.3, U2.4, U2.5, U2.6, U2.7, U2.8; no longer C1.-, C2.+, CV2_LEV.1, CV_2.P$1, Q2.B, U$1.3, U$1.4, U$1.5, U$1.6, U$1.7, U$1.8
- net N$12: now also RESONANCE.6
- net N$16: now also Q2.1; no longer Q2.C
- net N$21: now also Q1.2; no longer Q1.B
- net N$23: now also CV2.1, CV2_LEV.1; no longer CV2_LEV.3, CV_2.P$3
- net N$24: now also CV1_LEV.6
- net N$27: now also U2.13, U2.14; no longer U$1.13, U$1.14
- net N$3: now also Q1.1; no longer Q1.C
- net N$5: now also Q1.3, Q2.3; no longer Q1.E, Q2.E
Routing:
- net GND: track 436.0 -> 0.00 mm
- net +12V: track 188.2 -> 0.00 mm
- net -12V: track 139.4 -> 0.00 mm
- net N$16: track 92.3 -> 0.00 mm, vias 2 -> 0
- net N$21: track 80.2 -> 0.00 mm
- net N$27: track 80.1 -> 0.00 mm, vias 2 -> 0
- net N$14: track 60.4 -> 0.00 mm
- net N$6: track 45.9 -> 0.00 mm
- net N$9: track 41.4 -> 0.00 mm, vias 4 -> 0
- net N$12: track 40.0 -> 0.00 mm, vias 2 -> 0
- net N$24: track 34.7 -> 0.00 mm
- net N$1: track 33.6 -> 0.00 mm
- net N$10: track 31.5 -> 0.00 mm
- net N$11: track 30.9 -> 0.00 mm
- net N$20: track 28.4 -> 0.00 mm
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Other:
- board size 100.8 x 80 mm -> 100 x 80 mm

Commit message: decoupling caps
Parts:
- added C1, C10, C2, C4, C8, C9: 100n, rcl:C1206
Connections:
- net +12V: now also C1.1, C2.1, C4.1
- net -12V: now also C10.2, C8.2, C9.2
- net GND: now also C1.2, C10.1, C2.2, C4.2, C8.1, C9.1
Changed lines of the file:
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@@
 <element name="C24" library="rcl" package="C050-024X044" value="100n" x="22.86" y="-30.48"/>
 <element name="C25" library="rcl" package="C050-024X044" value="100n" x="3.81" y="-38.1"/>
+<element name="C1" library="rcl" package="C1206" value="100n" x="2.54" y="-44.45"/>
+<element name="C2" library="rcl" package="C1206" value="100n" x="2.54" y="-49.53"/>
+<element name="C4" library="rcl" package="C1206" value="100n" x="2.54" y="-54.61"/>
+<element name="C8" library="rcl" package="C1206" value="100n" x="2.54" y="-59.69"/>
+<element name="C9" library="rcl" package="C1206" value="100n" x="2.54" y="-64.77"/>
+<element name="C10" library="rcl" package="C1206" value="100n" x="2.54" y="-69.85"/>
 </elements>
 <signals>
@@
 <contactref element="FB4" pad="P$2"/>
 <contactref element="C25" pad="2"/>
+<contactref element="C8" pad="2"/>
+<contactref element="C9" pad="2"/>
+<contactref element="C10" pad="2"/>
 <wire x1="57.15" y1="40.64" x2="60.96" y2="53.34" width="0" layer="19" extent="1-1"/>
 <wire x1="48.26" y1="45.72" x2="57.15" y2="40.64" width="0" layer="19" extent="1-1"/>
@@
 <wire x1="16.47" y1="-31.75" x2="13.97" y2="-24.13" width="0" layer="19" extent="1-1"/>
 <wire x1="6.35" y1="-38.1" x2="16.47" y2="-31.75" width="0" layer="19" extent="1-1"/>
+<wire x1="3.94" y1="-59.69" x2="6.35" y2="-38.1" width="0" layer="19" extent="1-1"/>
+<wire x1="3.94" y1="-64.77" x2="3.94" y2="-59.69" width="0" layer="19" extent="1-1"/>
+<wire x1="3.94" y1="-69.85" x2="3.94" y2="-64.77" width="0" layer="19" extent="1-1"/>
 </signal>
 <signal name="+12V">
@@
 <contactref element="FB3" pad="P$2"/>
 <contactref element="C24" pad="1"/>
+<contactref element="C4" pad="1"/>
+<contactref element="C1" pad="1"/>
+<contactref element="C2" pad="1"/>
 <wire x1="76.2" y1="35.56" x2="68.58" y2="53.34" width="0" layer="19" extent="1-1"/>
 <wire x1="40.64" y1="53.34" x2="68.58" y2="53.34" width="0" layer="19" extent="1-1"/>
@@
 <wire x1="7.58" y1="-31.75" x2="20.32" y2="-30.48" width="0" layer="19" extent="1-1"/>
 <wire x1="1.27" y1="-24.13" x2="7.58" y2="-31.75" width="0" layer="19" extent="1-1"/>
+<wire x1="1.14" y1="-44.45" x2="7.58" y2="-31.75" width="0" layer="19" extent="1-1"/>
+<wire x1="1.14" y1="-49.53" x2="1.14" y2="-44.45" width="0" layer="19" extent="1-1"/>
+<wire x1="1.14" y1="-54.61" x2="1.14" y2="-49.53" width="0" layer="19" extent="1-1"/>
 </signal>
 <signal name="N$1">
@@
 <contactref element="U2" pad="6"/>
 <contactref element="U2" pad="5"/>
+<contactref element="C1" pad="2"/>
+<contactref element="C10" pad="1"/>
+<contactref element="C2" pad="2"/>
+<contactref element="C9" pad="1"/>
+<contactref element="C4" pad="2"/>
+<contactref element="C8" pad="1"/>
 <wire x1="83.82" y1="58.42" x2="83.82" y2="60.96" width="0" layer="19" extent="1-1"/>
 <wire x1="86.36" y1="57.15" x2="83.82" y2="58.42" width="0" layer="19" extent="1-1"/>
@@
 <wire x1="3.81" y1="-24.13" x2="11.43" y2="-24.13" width="0" layer="19" extent="1-1"/>
 <wire x1="1.27" y1="-38.1" x2="3.81" y2="-24.13" width="0" layer="19" extent="1-1"/>
+<wire x1="3.94" y1="-44.45" x2="1.27" y2="-38.1" width="0" layer="19" extent="1-1"/>
+<wire x1="3.94" y1="-49.53" x2="3.94" y2="-44.45" width="0" layer="19" extent="1-1"/>
+<wire x1="3.94" y1="-54.61" x2="3.94" y2="-49.53" width="0" layer="19" extent="1-1"/>
+<wire x1="1.14" y1="-59.69" x2="3.94" y2="-54.61" width="0" layer="19" extent="1-1"/>
+<wire x1="1.14" y1="-64.77" x2="1.14" y2="-59.69" width="0" layer="19" extent="1-1"/>
+<wire x1="1.14" y1="-69.85" x2="1.14" y2="-64.77" width="0" layer="19" extent="1-1"/>
 <wire x1="25.4" y1="-30.48" x2="11.43" y2="-24.13" width="0" layer="19" extent="1-1"/>
 <wire x1="39.37" y1="64.77" x2="45.72" y2="45.72" width="0" layer="19" extent="1-1"/>

Commit message: parts on the board
Parts:
- R1, R10, R11, R12, R13, R14, R15, R16, R17, R18, R19, R21, R4, R5, R6, R7, R8, R9: device rcl:0207/10 -> rcl:0207/7
- moved C10 123.7 mm to (67.3, 35.6), flipped to the bottom, turned to 270 degrees
- moved C9 117.7 mm to (83.8, 20.3), flipped to the bottom, turned to 90 degrees
- moved C2 112.3 mm to (83.8, 27.9), flipped to the bottom, turned to 90 degrees
- moved C1 97.1 mm to (67.3, 27.9), flipped to the bottom, turned to 270 degrees
- moved C8 93.7 mm to (44.5, 24.1), flipped to the bottom
- moved C4 85.9 mm to (36.8, 24.1), flipped to the bottom
- moved C25 68.9 mm to (10.2, 30.5), turned to 180 degrees
- moved FB3 67.5 mm to (24.1, 33.0), turned to 270 degrees
- moved FB4 65.4 mm to (5.08, 33.0), turned to 270 degrees
- moved C24 61.2 mm to (17.8, 30.5), turned to 180 degrees
- moved C22 60.4 mm to (17.8, 34.3), turned to 180 degrees
- moved C23 58.5 mm to (10.2, 34.3), turned to 180 degrees
- moved U2 57.2 mm to (15.2, 41.9)
- moved R17 33.8 mm to (78.2, 42.2), turned to 0 degrees
- moved R10 31.9 mm to (57.1, 39.4)
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Other:
- board size 100 x 80 mm -> 97.5 x 48.2 mm

Commit message: routed
Parts:
- moved R6 5.68 mm to (63.5, 20.3), turned to 180 degrees
- moved Q2 4.58 mm to (64.8, 15.2)
- moved Q1 4.58 mm to (61.0, 15.2)
- moved C9 1.27 mm to (83.8, 21.6), turned to 270 degrees
- moved C7 1.27 mm to (81.3, 13.3)
- moved R21 1.27 mm to (72.4, 11.4)
Routing:
- net -12V: track 0.00 -> 148.5 mm, vias 0 -> 1
- net +12V: track 0.00 -> 117.9 mm
- net N$16: track 0.00 -> 73.0 mm
- net N$19: track 0.00 -> 63.8 mm
- net N$21: track 0.00 -> 59.8 mm
- net N$26: track 0.00 -> 50.1 mm
- net N$14: track 0.00 -> 46.7 mm
- net N$9: track 0.00 -> 42.3 mm, vias 0 -> 1
- net N$3: track 0.00 -> 40.7 mm, vias 0 -> 1
- net N$27: track 0.00 -> 37.2 mm
- net N$6: track 0.00 -> 36.4 mm
- net N$12: track 0.00 -> 34.4 mm
- net N$24: track 0.00 -> 24.5 mm
- net N$1: track 0.00 -> 21.6 mm
- net N$2: track 0.00 -> 21.2 mm
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- added copper zone on layer 16, net GND
